Commit message: feat: working pub sub and spiky_star code

File: gazebo_models/spiky_star.urdf (robot description, URDF)
Before this commit: robot wall_star, 2 links, 1 joints
Links:
- link base_link: mass 1000.0 -> 10.0; geometry collision box size=0.375 0.0125 0.25; collision box size=0.375 0.0125 0.25
